File: hardware/Panel.sch (KiCad schematic (older format))
At the start: 18 parts, among them J101 Conn_01x02, J102 Header, J103 Header, J104 Conn_01x02, SW101 Rotary Encoder + Switch, SW102 10mm, SW103 10mm, SW104 B3W-9000-RG2N, U101 XC6206P, U102 ATtiny4313

Commit message: Rev2 fixes
- Move I2C pullups on main board
- Fix left/right/main buttons traces
Parts:
- added R102, R103: 10K, Resistor_SMD:R_0805_2012Metric_Pad1.20x1.40mm_HandSolder, symbol Device:R_Small
- SW102, SW103: symbol Switch:SW_Push -> Switch:SW_MEC_5E
- U101: footprint Package_TO_SOT_SMD:SOT-23 -> Package_TO_SOT_SMD:SOT-23_Handsoldering
- renumbered R102 to R104, R103 to R105
Connections:
- net labels added: MISO, MOSI, SCK
- wire segments 98 -> 113
Other:
- moved on the sheet: R104, R105, SW104, U102
