File: hardware/Oled Support.kicad_sch (KiCad schematic)
At the start: 13 parts, among them J201 Conn_01x02, J202 Conn_01x02

Commit message: Minor changes
Parts:
- gave numbers to parts that had none: 10
