File: hardware/Panel.kicad_pcb (KiCad board)
At the start: 2 copper layers, 65.3 x 64 mm, 33 parts, among them J101 Conn_01x02, J102 Header, J103 Header, J104 Conn_01x02, J201 Conn_01x02, J202 Conn_01x02, J203 SSD1306, SW101 Rotary Encoder + Switch, SW102 10mm, SW103 10mm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

Commit message: KiCad 7.0 update
Connections:
- net ~INT renamed ~{INT}
- net ~RST renamed ~{RST}
Other:
- net class Default removed
- board text added: "~{INT}"
- board text added: "~{RST}"
- board text removed: "~INT"
- board text removed: "~RST"

Commit message: Update to Kicad 8
Parts:
- BZ101: footprint Buzzer_Beeper:Buzzer_Murata_PKMCS0909E4000-R1 -> Buzzer_Beeper:Buzzer_Murata_PKMCS0909E
- J203: value SSD1306 -> SH1106
- U102: value ATtiny4313 -> ATtiny4313-S
Connections:
- J203 pad 7: (no net) -> unconnected-(J203-NC-Pad7)
- SW102 pad 2: GND -> LBTN
- SW103 pad 2: GND -> RBTN
- U102 pad 4: (no net) -> unconnected-(U102-PA1/XTAL2-Pad4)
Routing:
- net GND: track 100.6 -> 82.2 mm
- net VCC: track 78.8 -> 77.1 mm
- net SDA: track 97.2 -> 98.3 mm
- net LBTN: track 28.7 -> 28.1 mm
- net Net-(J203-VCC): track 8.24 -> 8.76 mm
